Commit message: v1.1.10

File: description/encoder.xacro (robot description, xacro)
@@ -1,32 +1,20 @@
 <?xml version="1.0"?>
-<robot xmlns:xacro="http://www.ros.org/wiki/xacro" name="encoder">
-    <gazebo>
-        <plugin name="encoder" filename="libgazebo_ros_diff_drive.so">
-            <ros>
-                <namespace>/</namespace>
-                <remapping>odom:=/odom</remapping>
-	        </ros>
-            <update_rate>30</update_rate>
-            <leftJoint>than_xe_banh_1</leftJoint>
-            <leftJoint>than_xe_banh_2</leftJoint>
-            <rightJoint>than_xe_banh_3</rightJoint>
-            <rightJoint>than_xe_banh_4</rightJoint>
-            <wheelSeparation>0.1566</wheelSeparation>
-            <wheelDiameter>0.07</wheelDiameter>
-	        <wheelAcceleration>1.0</wheelAcceleration>
-	        <wheelTorque>10</wheelTorque>
-            <!-- Chủ đề và khung TF -->
-	        <commandTopic>cmd_vel</commandTopic>
-	        <odometryTopic>odom</odometryTopic>
-	        <odometryFrame>odom</odometryFrame>
-	        <robotBaseFrame>base_footprint</robotBaseFrame>
-	        <!-- Xuất transform và trạng thái bánh xe -->
-	        <publishWheelTF>true</publishWheelTF>       	<!-- Xuất TF của bánh xe -->
-	        <publishOdomTF>true</publishOdomTF>         	<!-- Xuất TF của odometry -->
-	        <publishWheelJointState>true</publishWheelJointState> <!-- Xuất trạng thái joint của bánh xe -->
-	        <publishTf>1</publishTf>                    	<!-- Xuất thông tin TF -->
-        	<!-- Nguồn dữ liệu odometry (0 = ground truth, 1 = encoder) -->
-	        <odometrySource>encoder</odometrySource>
-	        <rosDebugLevel>info</rosDebugLevel>
-        </plugin>
+<robot xmlns:xacro="http://www.ros.org/wiki/xacro"  name="robot">
+	<gazebo>
+    	<plugin name="diff_drive" filename="libgazebo_ros_diff_drive.so">
+      		<leftJoint>than_xe_banh_1</leftJoint>
+      		<rightJoint>than_xe_banh_2</rightJoint>
+      		<wheelSeparation>0.35</wheelSeparation>
+      		<wheelDiameter>0.1</wheelDiameter>
+      		<maxWheelTorque>200</maxWheelTorque>
+      		<maxWheelAcceleration>10.0</maxWheelAcceleration>
+      		<commandTopic>cmd_vel</commandTopic>
+			<odometryTopic>odom</odometryTopic>
+			<odometryFrame>odom</odometryFrame>
+			<robotBaseFrame>than_xe</robotBaseFrame>
+      		<publish_odom>true</publish_odom>
+      		<publishOdomTF>true</publishOdomTF>
+      		<publishWheelTF>true</publishWheelTF>
+    	</plugin>
+  	</gazebo>
 </robot>

File: description/lidar.xacro (robot description, xacro)
@@ -18,5 +18,5 @@
                         <resolution>1.000000</resolution>
                         <min_angle>0.000000</min_angle>
-                        <max_angle>6.280000</max_angle>
+                        <max_angle>3.140000</max_angle>
                     </horizontal>
                 </scan>

File: description/xe_tang.urdf.xacro (robot description, xacro)
@@ -46,8 +46,4 @@
         </joint>
     </xacro:macro>
-    <xacro:include filename="camera.xacro"/>
-    <xacro:include filename="encoder.xacro"/>
-    <xacro:include filename="lidar.xacro"/>
-    <xacro:include filename="tay_may.xacro"/>
     <xacro:link link_name="than_xe"
                 x1="-0.234314" y1="0.0727514" z1="0.193682" roll1="0" pitch1="0" yaw1="0"
@@ -59,91 +55,8 @@
         <material>Gazebo/DarkGray</material>
     </gazebo>
-    <xacro:link link_name="banh_xe_1"
-                x1="-1.2677e-19" y1="4.67093e-18" z1="0.00430301" roll1="0" pitch1="0" yaw1="0"
-                mass="0.522006"
-                ixx="0.00049418" ixy="1.06373e-20" ixz="1.06547e-45" iyy="0.00049418" iyz="2.78846e-46" izz="0.000673955"
-                r="0.3" g="0.3" b="0.3" a="1.0"
-                x2="0" y2="0" z2="-0.025" roll2="-1.5708" pitch2="-3.64847e-42" yaw2="2.45344e-17"/>
-    <gazebo reference="banh_xe_1">
-        <material>Gazebo/Gray</material>
-    </gazebo>
-    <xacro:joint joint_name="than_xe_banh_1" type="revolute"
-                 x1="-0.365902" y1="0.212751" z1="0.169141" roll1="-1.5708" pitch1="1.42583" yaw1="3.14159"
-                 parent_link="than_xe"
-                 child_link="banh_xe_1"
-                 x2="0" y2="0" z2="1"
-                 effort="10" velocity="10" lower="-3.141592653589793" upper="3.141592653589793"/>
-    <xacro:link link_name="banh_xe_2"
-                x1="-1.2677e-19" y1="4.67093e-18" z1="0.00430301" roll1="0" pitch1="0" yaw1="0"
-                mass="0.522006"
-                ixx="0.00049418" ixy="2.78829e-20" ixz="9.04058e-46" iyy="0.00049418" iyz="-1.39449e-45" izz="0.000673955"
-                r="0.3" g="0.3" b="0.3" a="1.0"
-                x2="0" y2="0" z2="-0.025" roll2="-1.5708" pitch2="-1.90898e-42" yaw2="4.22367e-17"/>
-    <gazebo reference="banh_xe_2">
-        <material>Gazebo/Gray</material>
-    </gazebo>
-    <xacro:joint joint_name="than_xe_banh_2" type="revolute"
-                 x1="-0.105902" y1="0.212751" z1="0.169141" roll1="-1.5708" pitch1="1.05145" yaw1="3.14159"
-                 parent_link="than_xe"
-                 child_link="banh_xe_2"
-                 x2="0" y2="0" z2="1"
-                 effort="10" velocity="10" lower="-3.141592653589793" upper="3.141592653589793"/>
-    <xacro:link link_name="banh_xe_3"
-                x1="5.53844e-17" y1="4.67093e-18" z1="0.00430301" roll1="0" pitch1="0" yaw1="0"
-                mass="0.522006"
-                ixx="0.00049418" ixy="-1.19623e-20" ixz="0" iyy="0.00049418" iyz="0" izz="0.000673955"
-                r="0.3" g="0.3" b="0.3" a="1.0"
-                x2="5.55112e-17" y2="0" z2="-0.025" roll2="-1.5708" pitch2="0" yaw2="-1.73484e-17"/>
-    <gazebo reference="banh_xe_3">
-        <material>Gazebo/Gray</material>
-    </gazebo>
-    <xacro:joint joint_name="than_xe_banh_3" type="revolute"
-                 x1="-0.365902" y1="-0.0672486" z1="0.169141" roll1="-1.5708" pitch1="0.295982" yaw1="0"
-                 parent_link="than_xe"
-                 child_link="banh_xe_3"
-                 x2="0" y2="0" z2="1"
-                 effort="10" velocity="10" lower="-3.141592653589793" upper="3.141592653589793"/>
-    <xacro:link link_name="banh_xe_4"
-                x1="-1.2677e-19" y1="4.67093e-18" z1="0.00430301" roll1="0" pitch1="0" yaw1="0"
-                mass="0.522006"
-                ixx="0.00049418" ixy="1.49967e-21" ixz="6.65827e-46" iyy="0.00049418" iyz="-1.24813e-46" izz="0.000673955"
-                r="0.3" g="0.3" b="0.3" a="1.0"
-                x2="0" y2="0" z2="-0.025" roll2="-1.5708" pitch2="-2.12258e-42" yaw2="4.03777e-18"/>
-    <gazebo reference="banh_xe_4">
-        <material>Gazebo/Gray</material>
-    </gazebo>
-    <xacro:joint joint_name="than_xe_banh_4" type="revolute"
-                 x1="-0.105902" y1="-0.0672486" z1="0.169141" roll1="1.5708" pitch1="-1.53924" yaw1="3.14159"
-                 parent_link="than_xe"
-                 child_link="banh_xe_4"
-                 x2="0" y2="0" z2="1"
-                 effort="10" velocity="10" lower="-3.141592653589793" upper="3.141592653589793"/>
-    <xacro:link link_name="xich_1"
-                x1="2.74156e-16" y1="-4.8039e-17" z1="-0.03" roll1="0" pitch1="0" yaw1="0"
-                mass="2.81002"
-                ixx="0.00760602" ixy="1.11093e-06" ixz="0" iyy="0.0406757" iyz="0" izz="0.0465957"
-                r="0.1" g="0.1" b="0.1" a="1.0"
-                x2="3.33067e-16" y2="-5.55112e-17" z2="0" roll2="1.5708" pitch2="0" yaw2="0"/>
-    <gazebo reference="xich_1">
-        <material>Gazebo/FlatBlack</material>
-    </gazebo>
-    <xacro:joint joint_name="than_xe_xich_1" type="fixed"
-                 x1="-0.235839" y1="-0.0322486" z1="0.169009" roll1="-1.5708" pitch1="0" yaw1="0"
-                 parent_link="than_xe"
-                 child_link="xich_1"
-                 x2="0" y2="0" z2="1"/>
-    <xacro:link link_name="xich_2"
-                x1="-0.0432788" y1="-0.055" z1="-0.03" roll1="0" pitch1="0" yaw1="0"
-                mass="2.81002"
-                ixx="0.00760602" ixy="-1.11093e-06" ixz="0" iyy="0.0406757" iyz="0" izz="0.0465957"
-                r="0.1" g="0.1" b="0.1" a="1.0"
-                x2="-0.0432788" y2="-0.055" z2="-0.06" roll2="-1.5708" pitch2="0" yaw2="0"/>
-    <gazebo reference="xich_2">
-        <material>Gazebo/FlatBlack</material>
-    </gazebo>
-    <xacro:joint joint_name="than_xe_xich_2" type="fixed"
-                 x1="-0.278939" y1="0.177751" z1="0.114109" roll1="-1.5708" pitch1="0" yaw1="3.14159"
-                 parent_link="than_xe"
-                 child_link="xich_2"
-                 x2="0" y2="0" z2="1"/>
+    <xacro:include filename="arm_controller.xacro"/>
+    <xacro:include filename="base_controller.xacro"/>
+    <xacro:include filename="camera.xacro"/>
+    <xacro:include filename="encoder.xacro"/>
+    <xacro:include filename="lidar.xacro"/>
 </robot>
