Commit message: v1.1.2

File: description/camera.xacro (robot description, xacro)
@@ -8,4 +8,41 @@
     <gazebo reference="camera">
         <material>Gazebo/Green</material>
+        <sensor type="camera" name="camera_pi">
+            <update_rate>30.0</update_rate>
+            <camera name="head">
+                <horizontal_fov>1.3962634</horizontal_fov>
+                <image>
+                    <width>800</width>
+                    <height>800</height>
+                    <format>R8G8B8</format>
+                </image>
+                <clip>
+                    <near>0.02</near>
+                    <far>300</far>
+                </clip>
+                <noise>
+                    <type>gaussian</type>
+                    <!-- Noise is sampled independently per pixel on each frame.
+                    That pixel's noise value is added to each of its color
+                    channels, which at that point lie in the range [0,1]. -->
+                    <mean>0.0</mean>
+                    <stddev>0.007</stddev>
+                </noise>
+            </camera>
+            <plugin name="camera_controller" filename="libgazebo_ros_camera.so">
+                <alwaysOn>true</alwaysOn>
+                <updateRate>0.0</updateRate>
+                <cameraName>rrbot/camera1</cameraName>
+                <imageTopicName>image_raw</imageTopicName>
+                <cameraInfoTopicName>camera_info</cameraInfoTopicName>
+                <frameName>camera_link</frameName>
+                <hackBaseline>0.07</hackBaseline>
+                <distortionK1>0.0</distortionK1>
+                <distortionK2>0.0</distortionK2>
+                <distortionK3>0.0</distortionK3>
+                <distortionT1>0.0</distortionT1>
+                <distortionT2>0.0</distortionT2>
+            </plugin>
+        </sensor>
     </gazebo>
     <xacro:joint joint_name="than_xe_camera" type="fixed"

File: description/macros.xacro (robot description, xacro)
@@ -17,5 +17,7 @@
                     <mesh filename="package://xe_tang/meshes/${link_name}.stl"/>
                 </geometry>
-                <material name="${link_name}_material"/>
+                <material name="${link_name}_material">
+                    <color rgba="0 0 0 1.0"/>
+                </material>
             </visual>
             <collision>

File: description/xe_tang.urdf.xacro (robot description, xacro)
@@ -4,4 +4,5 @@
     <xacro:include filename="camera.xacro"/>
     <xacro:include filename="lidar.xacro"/>
+    <xacro:include filename="tay_may.xacro"/>
     <xacro:link link_name="than_xe"
                 x1="-0.234314" y1="0.0727514" z1="0.193682" roll1="0" pitch1="0" yaw1="0"
@@ -94,44 +95,3 @@
                  child_link="xich_2"
                  x2="0" y2="0" z2="1"/>
-    <xacro:link link_name="khau_1"
-                x1="-1.96426e-19" y1="-3.3125e-18" z1="-0.186482" roll1="0" pitch1="0" yaw1="0"
-                mass="1.23111"
-                ixx="0.0507892" ixy="0" ixz="0" iyy="0.0507892" iyz="0" izz="0.00254127"
-                x2="0" y2="0" z2="0" roll2="3.14159" pitch2="0" yaw2="0"/>
-    <gazebo reference="khau_1">
-        <material>Gazebo/White</material>
-    </gazebo>
-    <xacro:joint joint_name="than_xe_khau_1" type="fixed"
-                 x1="-0.173402" y1="0.0727514" z1="0.243141" roll1="3.14159" pitch1="0" yaw1="0"
-                 parent_link="than_xe"
-                 child_link="khau_1"
-                 x2="0" y2="0" z2="1"/>
-    <xacro:link link_name="khop"
-                x1="7.82984e-19" y1="4.06082e-18" z1="-0.015" roll1="0" pitch1="0" yaw1="0"
-                mass="0.485965"
-                ixx="0.000545572" ixy="0" ixz="0" iyy="0.000545572" iyz="0" izz="0.00101825"
-                x2="0" y2="0" z2="-0.03" roll2="0" pitch2="0" yaw2="0"/>
-    <gazebo reference="khop">
-        <material>Gazebo/SkyBlue</material>
-    </gazebo>
-    <xacro:joint joint_name="khau_1_khop" type="prismatic"
-                 x1="0" y1="0" z1="-0.187558" roll1="3.14159" pitch1="0" yaw1="-1.86886e-29"
-                 parent_link="khau_1"
-                 child_link="khop"
-                 x2="0" y2="0" z2="1"
-                 effort="10" velocity="10" lower="-0.112558" upper="0.257442"/>
-    <xacro:link link_name="khau_2"
-                x1="0.228819" y1="-6.22477e-10" z1="-0.0150176" roll1="0" pitch1="0" yaw1="0"
-                mass="1.61532"
-                ixx="0.0023024" ixy="-2.36835e-10" ixz="-6.71781e-06" iyy="0.0271882" iyz="1.68742e-11" izz="0.0288969"
-                x2="0" y2="0" z2="-0.03" roll2="-1.81353e-41" pitch2="1.58254e-41" yaw2="6.17393e-18"/>
-    <gazebo reference="khau_2">
-        <material>Gazebo/White</material>
-    </gazebo>
-    <xacro:joint joint_name="khop_khau_2" type="revolute"
-                 x1="-8.32667e-17" y1="5.55112e-17" z1="0" roll1="-1.81771e-25" pitch1="5.10563e-25" yaw1="-0.72926"
-                 parent_link="khop"
-                 child_link="khau_2"
-                 x2="0" y2="0" z2="1"
-                 effort="10" velocity="10" lower="-3.141592653589793" upper="3.141592653589793"/>
 </robot>

Commit message: v1.1.4

File: description/camera.xacro (robot description, xacro)
@@ -5,10 +5,11 @@
                 mass="0.00147364"
                 ixx="7.56624e-08" ixy="0" ixz="0" iyy="7.05662e-08" iyz="-2.12341e-09" izz="1.43344e-07"
+                r="0" g="1.0" b="0" a="1.0"
                 x2="0" y2="0" z2="0" roll2="3.14159" pitch2="0" yaw2="0"/>
     <gazebo reference="camera">
         <material>Gazebo/Green</material>
-        <sensor type="camera" name="camera_pi">
+        <sensor type="camera" name="backup_camera">
             <update_rate>30.0</update_rate>
-            <camera name="head">
+            <camera name="camera_pi">
                 <horizontal_fov>1.3962634</horizontal_fov>
                 <image>
@@ -23,7 +24,4 @@
                 <noise>
                     <type>gaussian</type>
-                    <!-- Noise is sampled independently per pixel on each frame.
-                    That pixel's noise value is added to each of its color
-                    channels, which at that point lie in the range [0,1]. -->
                     <mean>0.0</mean>
                     <stddev>0.007</stddev>
@@ -33,8 +31,8 @@
                 <alwaysOn>true</alwaysOn>
                 <updateRate>0.0</updateRate>
-                <cameraName>rrbot/camera1</cameraName>
+                <cameraName>camera_pi</cameraName>
                 <imageTopicName>image_raw</imageTopicName>
                 <cameraInfoTopicName>camera_info</cameraInfoTopicName>
-                <frameName>camera_link</frameName>
+                <frameName>camera</frameName>
                 <hackBaseline>0.07</hackBaseline>
                 <distortionK1>0.0</distortionK1>

File: description/lidar.xacro (robot description, xacro)
@@ -5,4 +5,5 @@
                 mass="0.0941187"
                 ixx="3.50997e-05" ixy="-3.88943e-23" ixz="5.54226e-07" iyy="2.94944e-05" iyz="-3.84572e-24" izz="5.46193e-05"
+                r="0" g="0" b="0" a="1.0"
                 x2="-5.55112e-17" y2="-6.93889e-17" z2="-2.77556e-17" roll2="3.14159" pitch2="0" yaw2="-6.93889e-18"/>
     <gazebo reference="lidar">

File: description/tay_may.xacro (robot description, xacro)
@@ -5,4 +5,5 @@
                 mass="1.23111"
                 ixx="0.0507892" ixy="0" ixz="0" iyy="0.0507892" iyz="0" izz="0.00254127"
+                r="1.0" g="1.0" b="1.0" a="1.0"
                 x2="0" y2="0" z2="0" roll2="3.14159" pitch2="0" yaw2="0"/>
     <gazebo reference="khau_1">
@@ -18,4 +19,5 @@
                 mass="0.485965"
                 ixx="0.000545572" ixy="0" ixz="0" iyy="0.000545572" iyz="0" izz="0.00101825"
+                r="0.13" g="0.44" b="0.70" a="1.0"
                 x2="0" y2="0" z2="-0.03" roll2="0" pitch2="0" yaw2="0"/>
     <gazebo reference="khop">
@@ -32,4 +34,5 @@
                 mass="1.61532"
                 ixx="0.0023024" ixy="-2.36835e-10" ixz="-6.71781e-06" iyy="0.0271882" iyz="1.68742e-11" izz="0.0288969"
+                r="1.0" g="1.0" b="1.0" a="1.0"
                 x2="0" y2="0" z2="-0.03" roll2="-1.81353e-41" pitch2="1.58254e-41" yaw2="6.17393e-18"/>
     <gazebo reference="khau_2">

File: description/xe_tang.urdf.xacro (robot description, xacro)
@@ -1,5 +1,49 @@
 <?xml version="1.0"?>
 <robot xmlns:xacro="http://www.ros.org/wiki/xacro" name="xe-tang">
-    <xacro:include filename="macros.xacro"/>
+    <xacro:macro name="link" params="link_name
+                                     x1 y1 z1 roll1 pitch1 yaw1
+                                     mass
+                                     ixx ixy ixz iyy iyz izz
+                                     r g b a
+                                     x2 y2 z2 roll2 pitch2 yaw2">
+        <link name="${link_name}">
+            <inertial>
+                <origin xyz="${x1} ${y1} ${z1}" rpy="${roll1} ${pitch1} ${yaw1}"/>
+                <mass value="${mass}"/>
+                <inertia ixx="${ixx}" ixy="${ixy}" ixz="${ixz}" iyy="${iyy}" iyz="${iyz}" izz="${izz}"/>
+            </inertial>
+            <visual>
+                <origin xyz="${x2} ${y2} ${z2}" rpy="${roll2} ${pitch2} ${yaw2}"/>
+                <geometry>
+                    <mesh filename="package://xe_tang/meshes/${link_name}.stl"/>
+                </geometry>
+                <material name="${link_name}_material">
+                    <color rgba="${r} ${g} ${b} ${a}"/>
+                </material>
+            </visual>
+            <collision>
+                <origin xyz="${x2} ${y2} ${z2}" rpy="${roll2} ${pitch2} ${yaw2}"/>
+                <geometry>
+                    <mesh filename="package://xe_tang/meshes/${link_name}.stl"/>
+                </geometry>
+            </collision>
+        </link>
+    </xacro:macro>
+    <xacro:macro name="joint" params="joint_name type
+                                      x1 y1 z1 roll1 pitch1 yaw1
+                                      parent_link
+                                      child_link
+                                      x2 y2 z2
+                                      effort:=0 velocity:=0 lower:=0 upper:=0">
+        <joint name="${joint_name}" type="${type}">
+            <origin xyz="${x1} ${y1} ${z1}" rpy="${roll1} ${pitch1} ${yaw1}"/>
+            <parent link="${parent_link}"/>
+            <child link="${child_link}"/>
+            <axis xyz="${x2} ${y2} ${z2}"/>
+            <xacro:if value="${type == 'revolute' or type == 'prismatic'}">
+                <limit effort="${effort}" velocity="${velocity}" lower="${lower}" upper="${upper}"/>
+            </xacro:if>
+        </joint>
+    </xacro:macro>
     <xacro:include filename="camera.xacro"/>
     <xacro:include filename="lidar.xacro"/>
@@ -9,4 +53,5 @@
                 mass="7.43294"
                 ixx="0.0323519" ixy="0" ixz="-0.000431382" iyy="0.0606346" iyz="0" izz="0.0810268"
+                r="0.175" g="0.175" b="0.175" a="1.0"
                 x2="-0.235902" y2="0.0727514" z2="0.144141" roll2="0" pitch2="0" yaw2="0"/>
     <gazebo reference="than_xe">
@@ -17,4 +62,5 @@
                 mass="0.522006"
                 ixx="0.00049418" ixy="1.06373e-20" ixz="1.06547e-45" iyy="0.00049418" iyz="2.78846e-46" izz="0.000673955"
+                r="0.3" g="0.3" b="0.3" a="1.0"
                 x2="0" y2="0" z2="-0.025" roll2="-1.5708" pitch2="-3.64847e-42" yaw2="2.45344e-17"/>
     <gazebo reference="banh_xe_1">
@@ -31,4 +77,5 @@
                 mass="0.522006"
                 ixx="0.00049418" ixy="2.78829e-20" ixz="9.04058e-46" iyy="0.00049418" iyz="-1.39449e-45" izz="0.000673955"
+                r="0.3" g="0.3" b="0.3" a="1.0"
                 x2="0" y2="0" z2="-0.025" roll2="-1.5708" pitch2="-1.90898e-42" yaw2="4.22367e-17"/>
     <gazebo reference="banh_xe_2">
@@ -45,4 +92,5 @@
                 mass="0.522006"
                 ixx="0.00049418" ixy="-1.19623e-20" ixz="0" iyy="0.00049418" iyz="0" izz="0.000673955"
+                r="0.3" g="0.3" b="0.3" a="1.0"
                 x2="5.55112e-17" y2="0" z2="-0.025" roll2="-1.5708" pitch2="0" yaw2="-1.73484e-17"/>
     <gazebo reference="banh_xe_3">
@@ -59,4 +107,5 @@
                 mass="0.522006"
                 ixx="0.00049418" ixy="1.49967e-21" ixz="6.65827e-46" iyy="0.00049418" iyz="-1.24813e-46" izz="0.000673955"
+                r="0.3" g="0.3" b="0.3" a="1.0"
                 x2="0" y2="0" z2="-0.025" roll2="-1.5708" pitch2="-2.12258e-42" yaw2="4.03777e-18"/>
     <gazebo reference="banh_xe_4">
@@ -73,4 +122,5 @@
                 mass="2.81002"
                 ixx="0.00760602" ixy="1.11093e-06" ixz="0" iyy="0.0406757" iyz="0" izz="0.0465957"
+                r="0.1" g="0.1" b="0.1" a="1.0"
                 x2="3.33067e-16" y2="-5.55112e-17" z2="0" roll2="1.5708" pitch2="0" yaw2="0"/>
     <gazebo reference="xich_1">
@@ -86,4 +136,5 @@
                 mass="2.81002"
                 ixx="0.00760602" ixy="-1.11093e-06" ixz="0" iyy="0.0406757" iyz="0" izz="0.0465957"
+                r="0.1" g="0.1" b="0.1" a="1.0"
                 x2="-0.0432788" y2="-0.055" z2="-0.06" roll2="-1.5708" pitch2="0" yaw2="0"/>
     <gazebo reference="xich_2">

Commit message: v1.1.5. camera.xacro

File: description/camera.xacro (robot description, xacro)
@@ -7,9 +7,23 @@
                 r="0" g="1.0" b="0" a="1.0"
                 x2="0" y2="0" z2="0" roll2="3.14159" pitch2="0" yaw2="0"/>
+    <link name="camera_optical">
+        <inertial>
+                <origin xyz="-1.08316e-18 -0.000645903 -0.00126913" rpy="0 0 0"/>
+                <mass value="0.00000000001"/>
+                <inertia ixx="7.56624e-08" ixy="0" ixz="0" iyy="7.05662e-08" iyz="-2.12341e-09" izz="1.43344e-07"/>
+            </inertial>
+        <visual>
+            <geometry>
+                <box size="0.00000000001 0.00000000001 0.00000000001"/>
+            </geometry>
+        </visual>
+    </link>
     <gazebo reference="camera">
         <material>Gazebo/Green</material>
-        <sensor type="camera" name="backup_camera">
+    </gazebo>
+    <gazebo reference="camera_optical">
+        <sensor name="camera" type="camera">
             <update_rate>30.0</update_rate>
-            <camera name="camera_pi">
+            <camera>
                 <horizontal_fov>1.3962634</horizontal_fov>
                 <image>
@@ -34,5 +48,5 @@
                 <imageTopicName>image_raw</imageTopicName>
                 <cameraInfoTopicName>camera_info</cameraInfoTopicName>
-                <frameName>camera</frameName>
+                <frameName>camera_optical</frameName>
                 <hackBaseline>0.07</hackBaseline>
                 <distortionK1>0.0</distortionK1>
@@ -49,3 +63,8 @@
                  child_link="camera"
                  x2="0" y2="0" z2="1"/>
+    <xacro:joint joint_name="camera_camera_optical" type="fixed"
+                 x1="0" y1="0" z1="0" roll1="1.5708" pitch1="1.5708" yaw1="0"
+                 parent_link="camera"
+                 child_link="camera_optical"
+                 x2="0" y2="0" z2="1"/>
 </robot>

Commit message: v1.2.1

File: description/camera.xacro (robot description, xacro)
@@ -7,16 +7,5 @@
                 r="0" g="1.0" b="0" a="1.0"
                 x2="0" y2="0" z2="0" roll2="3.14159" pitch2="0" yaw2="0"/>
-    <link name="camera_optical">
-        <inertial>
-                <origin xyz="-1.08316e-18 -0.000645903 -0.00126913" rpy="0 0 0"/>
-                <mass value="0.00000000001"/>
-                <inertia ixx="7.56624e-08" ixy="0" ixz="0" iyy="7.05662e-08" iyz="-2.12341e-09" izz="1.43344e-07"/>
-            </inertial>
-        <visual>
-            <geometry>
-                <box size="0.00000000001 0.00000000001 0.00000000001"/>
-            </geometry>
-        </visual>
-    </link>
+    <link name="camera_optical"/>
     <gazebo reference="camera">
         <material>Gazebo/Green</material>
