Commit message: v1.2.2

File: description/xe_tang.urdf.xacro (robot description, xacro)
@@ -46,5 +46,4 @@
         </joint>
     </xacro:macro>
-    <link name="world"/>
     <xacro:link link_name="than_xe"
                 x1="-0.234314" y1="0.0727514" z1="0.193682" roll1="0" pitch1="0" yaw1="0"
@@ -53,4 +52,5 @@
                 r="0.175" g="0.175" b="0.175" a="1.0"
                 x2="-0.235902" y2="0.0727514" z2="0.144141" roll2="0" pitch2="0" yaw2="0"/>
+    <link name="world"/>
     <gazebo reference="than_xe">
         <material>Gazebo/DarkGray</material>
@@ -63,5 +63,4 @@
     <xacro:include filename="base_controller.xacro"/>
     <xacro:include filename="camera.xacro"/>
-    <xacro:include filename="encoder.xacro"/>
     <xacro:include filename="lidar.xacro"/>
 </robot>

Commit message: v1.3.5

File: description/xe_tang.urdf.xacro (robot description, xacro)
@@ -53,5 +53,4 @@
                 r="0.175" g="0.175" b="0.175" a="1.0"
                 x2="0.00243663" y2="4.16334e-17" z2="0.0391321" roll2="0" pitch2="0" yaw2="0"/>
-    <link name="world"/>
     <gazebo reference="than_xe">
         <material>Gazebo/DarkGray</material>
@@ -59,8 +58,4 @@
         <mu2>0.2</mu2>
     </gazebo>
-    <xacro:joint joint_name="world_than_xe" type="fixed"
-                 x1="0" y1="0" z1="0" roll1="0" pitch1="0" yaw1="0"
-                 parent_link="world"
-                 child_link="than_xe"/>
     <xacro:include filename="arm_controller.xacro"/>
     <xacro:include filename="base_controller.xacro"/>
