Commit message: v1.3.1

File: description/base_controller.xacro (robot description, xacro)
@@ -87,27 +87,27 @@
                  parent_link="than_xe"
                  child_link="xich_2"/>
-    <transmission name="tran_left_wheel">
-        <type>transmission_interface/SimpleTransmission</type>
-        <joint name="than_xe_banh_1">
-        <hardwareInterface>hardware_interface/VelocityJointInterface</hardwareInterface>
-        </joint>
-        <actuator name="left_wheel_motor">
-        <hardwareInterface>hardware_interface/VelocityJointInterface</hardwareInterface>
-        <mechanicalReduction>1</mechanicalReduction>
-        </actuator>
-    </transmission>
     <transmission name="tran_right_wheel">
         <type>transmission_interface/SimpleTransmission</type>
         <joint name="than_xe_banh_2">
-        <hardwareInterface>hardware_interface/VelocityJointInterface</hardwareInterface>
+            <hardwareInterface>hardware_interface/VelocityJointInterface</hardwareInterface>
         </joint>
         <actuator name="right_wheel_motor">
-        <hardwareInterface>hardware_interface/VelocityJointInterface</hardwareInterface>
-        <mechanicalReduction>1</mechanicalReduction>
+            <hardwareInterface>hardware_interface/VelocityJointInterface</hardwareInterface>
+            <mechanicalReduction>1</mechanicalReduction>
+        </actuator>
+    </transmission>
+    <transmission name="tran_left_wheel">
+        <type>transmission_interface/SimpleTransmission</type>
+        <joint name="than_xe_banh_4">
+            <hardwareInterface>hardware_interface/VelocityJointInterface</hardwareInterface>
+        </joint>
+        <actuator name="left_wheel_motor">
+            <hardwareInterface>hardware_interface/VelocityJointInterface</hardwareInterface>
+            <mechanicalReduction>1</mechanicalReduction>
         </actuator>
     </transmission>
     <gazebo>
         <plugin name="gazebo_ros_control" filename="libgazebo_ros_control.so">
-        <robotNamespace>/xe_tang</robotNamespace>
+            <robotNamespace>/xe_tang</robotNamespace>
         </plugin>
     </gazebo>

Commit message: v1.3.2

File: description/base_controller.xacro (robot description, xacro)
@@ -15,5 +15,5 @@
                  child_link="banh_xe_1"
                  x2="0" y2="0" z2="1"
-                 effort="10" velocity="10" lower="-3.141592653589793" upper="3.141592653589793"/>
+                 effort="10" velocity="10" lower="-${PI}" upper="${PI}"/>
     <xacro:link link_name="banh_xe_2"
                 x1="-1.63473e-19" y1="-9.18731e-18" z1="0.00430301" roll1="0" pitch1="0" yaw1="0"
@@ -30,5 +30,5 @@
                  child_link="banh_xe_2"
                  x2="0" y2="0" z2="1"
-                 effort="10" velocity="10" lower="-3.141592653589793" upper="3.141592653589793"/>
+                 effort="10" velocity="10" lower="-${PI}" upper="${PI}"/>
     <xacro:link link_name="banh_xe_3"
                 x1="-1.63473e-19" y1="8.15992e-18" z1="0.00430301" roll1="0" pitch1="0" yaw1="0"
@@ -45,5 +45,5 @@
                  child_link="banh_xe_3"
                  x2="0" y2="0" z2="1"
-                 effort="10" velocity="10" lower="-3.141592653589793" upper="3.141592653589793"/>
+                 effort="10" velocity="10" lower="-${PI}" upper="${PI}"/>
     <xacro:link link_name="banh_xe_4"
                 x1="2.75921e-17" y1="4.69047e-18" z1="0.00430301" roll1="0" pitch1="0" yaw1="0"
@@ -60,5 +60,5 @@
                  child_link="banh_xe_4"
                  x2="0" y2="0" z2="1"
-                 effort="10" velocity="10" lower="-3.141592653589793" upper="3.141592653589793"/>
+                 effort="10" velocity="10" lower="-${PI}" upper="${PI}"/>
     <xacro:link link_name="xich_1"
                 x1="3.10096e-16" y1="-4.79297e-17" z1="-0.03" roll1="0" pitch1="0" yaw1="0"
@@ -87,28 +87,28 @@
                  parent_link="than_xe"
                  child_link="xich_2"/>
+    <gazebo>
+        <plugin name="gazebo_ros_control" filename="libgazebo_ros_control.so">
+            <robotNamespace>xe_tang</robotNamespace>
+        </plugin>
+    </gazebo>
+    <transmission name="tran_left_wheel">
+        <type>transmission_interface/SimpleTransmission</type>
+        <joint name="than_xe_banh_4">
+            <hardwareInterface>hardware_interface/EffortJointInterface</hardwareInterface>
+        </joint>
+        <actuator name="left_wheel_motor">
+            <hardwareInterface>hardware_interface/EffortJointInterface</hardwareInterface>
+            <mechanicalReduction>1</mechanicalReduction>
+        </actuator>
+    </transmission>
     <transmission name="tran_right_wheel">
         <type>transmission_interface/SimpleTransmission</type>
         <joint name="than_xe_banh_2">
-            <hardwareInterface>hardware_interface/VelocityJointInterface</hardwareInterface>
+            <hardwareInterface>hardware_interface/EffortJointInterface</hardwareInterface>
         </joint>
         <actuator name="right_wheel_motor">
-            <hardwareInterface>hardware_interface/VelocityJointInterface</hardwareInterface>
+            <hardwareInterface>hardware_interface/EffortJointInterface</hardwareInterface>
             <mechanicalReduction>1</mechanicalReduction>
         </actuator>
     </transmission>
-    <transmission name="tran_left_wheel">
-        <type>transmission_interface/SimpleTransmission</type>
-        <joint name="than_xe_banh_4">
-            <hardwareInterface>hardware_interface/VelocityJointInterface</hardwareInterface>
-        </joint>
-        <actuator name="left_wheel_motor">
-            <hardwareInterface>hardware_interface/VelocityJointInterface</hardwareInterface>
-            <mechanicalReduction>1</mechanicalReduction>
-        </actuator>
-    </transmission>
-    <gazebo>
-        <plugin name="gazebo_ros_control" filename="libgazebo_ros_control.so">
-            <robotNamespace>/xe_tang</robotNamespace>
-        </plugin>
-    </gazebo>
 </robot>

File: description/xe_tang.urdf.xacro (robot description, xacro)
@@ -46,4 +46,5 @@
         </joint>
     </xacro:macro>
+    <xacro:property name="PI" value="3.141592653589793"/>
     <xacro:link link_name="than_xe"
                 x1="0.00402455" y1="4.22475e-17" z1="0.0886727" roll1="0" pitch1="0" yaw1="0"

Commit message: v1.3.6

File: description/base_controller.xacro (robot description, xacro)
@@ -100,53 +100,19 @@
                  child_link="xich_2"/>
     <gazebo>
-        <plugin name="gazebo_ros_control" filename="libgazebo_ros_control.so">
-            <robotNamespace>/xe_tang</robotNamespace>
-        </plugin>
-    </gazebo>
-    <transmission name="tran_left_wheel">
-        <type>transmission_interface/SimpleTransmission</type>
-        <joint name="than_xe_banh_4">
-            <hardwareInterface>hardware_interface/EffortJointInterface</hardwareInterface>
-        </joint>
-        <actuator name="left_wheel_motor">
-            <hardwareInterface>hardware_interface/EffortJointInterface</hardwareInterface>
-            <mechanicalReduction>1</mechanicalReduction>
-        </actuator>
-    </transmission>
-    <transmission name="tran_right_wheel">
-        <type>transmission_interface/SimpleTransmission</type>
-        <joint name="than_xe_banh_2">
-            <hardwareInterface>hardware_interface/EffortJointInterface</hardwareInterface>
-        </joint>
-        <actuator name="right_wheel_motor">
-            <hardwareInterface>hardware_interface/EffortJointInterface</hardwareInterface>
-            <mechanicalReduction>1</mechanicalReduction>
-        </actuator>
-    </transmission>
-    <gazebo>
-        <plugin name="diff_drive" filename="libgazebo_ros_diff_drive.so">
-            <ros>
-                <robotNamespace>/xe_tang</robotNamespace>
-            </ros>
-            <numWheelPairs>1</numWheelPairs>
+        <plugin name='diff_drive' filename='libgazebo_ros_diff_drive.so'>
+            <updateRate>50</updateRate>
             <leftJoint>than_xe_banh_4</leftJoint>
-      		<rightJoint>than_xe_banh_2</rightJoint>
-      		<wheelSeparation>0.135</wheelSeparation>
-      		<wheelDiameter>0.1</wheelDiameter>
-      		<maxWheelTorque>200</maxWheelTorque>
-      		<maxWheelAcceleration>10.0</maxWheelAcceleration>
-      		<commandTopic>cmd_vel</commandTopic>
-			<odometryTopic>odom</odometryTopic>
-			<odometryFrame>odom</odometryFrame>
-			<robotBaseFrame>than_xe</robotBaseFrame>
-			<publishTf>true</publishTf>
-      		<publishOdomTF>true</publishOdomTF>
-      		<publishWheelTF>true</publishWheelTF>
-			<rosDebugLevel>INFO</rosDebugLevel>
-			<publishWheelJointState>true</publishWheelJointState>
-			<wheelAcceleration>1.0</wheelAcceleration>
-			<wheelTorque>10</wheelTorque>
-			<updateRate>100</updateRate>
-			<odometrySource>encoder</odometrySource>
+            <rightJoint>than_xe_banh_2</rightJoint>
+            <wheelSeparation>0.135</wheelSeparation>
+            <wheelDiameter>0.1</wheelDiameter>
+            <commandTopic>cmd_vel</commandTopic>
+            <odometryTopic>odom</odometryTopic>
+            <odometryFrame>odom</odometryFrame>
+            <robotBaseFrame>than_xe</robotBaseFrame>
+            <odometrySource>0</odometrySource>
+            <publishWheelTF>true</publishWheelTF>
+            <publishOdom>true</publishOdom>
+            <publishWheelJointState>true</publishWheelJointState>
+            <legacyMode>false</legacyMode>
         </plugin>
     </gazebo>

Commit message: continuous

File: description/base_controller.xacro (robot description, xacro)
@@ -12,10 +12,10 @@
         <mu2>0.2</mu2>
     </gazebo>
-    <xacro:joint joint_name="than_xe_banh_1" type="revolute"
+    <xacro:joint joint_name="than_xe_banh_1" type="continuous"
                  x1="-0.127563" y1="0.14" z1="0.0641321" roll1="-1.5708" pitch1="1.42583" yaw1="3.14159"
                  parent_link="than_xe"
                  child_link="banh_xe_1"
                  x2="0" y2="0" z2="1"
-                 effort="10" velocity="10" lower="-${PI}" upper="${PI}"/>
+                 effort="10" velocity="10"/>
     <xacro:link link_name="banh_xe_2"
                 x1="-1.63473e-19" y1="-9.18731e-18" z1="0.00430301" roll1="0" pitch1="0" yaw1="0"
@@ -29,10 +29,10 @@
         <mu2>0.2</mu2>
     </gazebo>
-    <xacro:joint joint_name="than_xe_banh_2" type="revolute"
+    <xacro:joint joint_name="than_xe_banh_2" type="continuous"
                  x1="0.132437" y1="0.14" z1="0.0641321" roll1="-1.5708" pitch1="1.05145" yaw1="3.14159"
                  parent_link="than_xe"
                  child_link="banh_xe_2"
                  x2="0" y2="0" z2="1"
-                 effort="10" velocity="10" lower="-${PI}" upper="${PI}"/>
+                 effort="10" velocity="10"/>
     <xacro:link link_name="banh_xe_3"
                 x1="-1.63473e-19" y1="8.15992e-18" z1="0.00430301" roll1="0" pitch1="0" yaw1="0"
@@ -46,10 +46,10 @@
         <mu2>0.2</mu2>
     </gazebo>
-    <xacro:joint joint_name="than_xe_banh_3" type="revolute"
+    <xacro:joint joint_name="than_xe_banh_3" type="continuous"
                  x1="-0.127563" y1="-0.14" z1="0.0641321" roll1="-1.5708" pitch1="0.295982" yaw1="0"
                  parent_link="than_xe"
                  child_link="banh_xe_3"
                  x2="0" y2="0" z2="1"
-                 effort="10" velocity="10" lower="-${PI}" upper="${PI}"/>
+                 effort="10" velocity="10"/>
     <xacro:link link_name="banh_xe_4"
                 x1="2.75921e-17" y1="4.69047e-18" z1="0.00430301" roll1="0" pitch1="0" yaw1="0"
@@ -63,10 +63,10 @@
         <mu2>0.2</mu2>
     </gazebo>
-    <xacro:joint joint_name="than_xe_banh_4" type="revolute"
+    <xacro:joint joint_name="than_xe_banh_4" type="continuous"
                  x1="0.132437" y1="-0.14" z1="0.0641321" roll1="1.5708" pitch1="0.033338" yaw1="3.14159"
                  parent_link="than_xe"
                  child_link="banh_xe_4"
                  x2="0" y2="0" z2="1"
-                 effort="10" velocity="10" lower="-${PI}" upper="${PI}"/>
+                 effort="10" velocity="10"/>
     <xacro:link link_name="xich_1"
                 x1="3.10096e-16" y1="-4.79297e-17" z1="-0.03" roll1="0" pitch1="0" yaw1="0"

File: description/xe_tang.urdf.xacro (robot description, xacro)
@@ -44,4 +44,8 @@
                 <limit effort="${effort}" velocity="${velocity}" lower="${lower}" upper="${upper}"/>
             </xacro:if>
+            <xacro:if value="${type == 'continuous'}">
+                <axis xyz="${x2} ${y2} ${z2}"/>
+                <limit effort="${effort}" velocity="${velocity}"/>
+            </xacro:if>
         </joint>
     </xacro:macro>

Commit message: v.1.3.7

File: description/base_controller.xacro (robot description, xacro)
@@ -7,9 +7,5 @@
                 r="0.3" g="0.3" b="0.3" a="1.0"
                 x2="-6.93889e-18" y2="2.77556e-17" z2="-0.025" roll2="-1.5708" pitch2="-3.64847e-42" yaw2="2.45344e-17"/>
-    <gazebo reference="banh_xe_1">
-        <material>Gazebo/Gray</material>
-        <mu1>0.2</mu1>
-        <mu2>0.2</mu2>
-    </gazebo>
+    <xacro:gazebo reference="banh_xe_1" material="Gazebo/Gray" mu1="0.2" mu2="0.2"/>
     <xacro:joint joint_name="than_xe_banh_1" type="continuous"
                  x1="-0.127563" y1="0.14" z1="0.0641321" roll1="-1.5708" pitch1="1.42583" yaw1="3.14159"
@@ -24,9 +20,5 @@
                 r="0.3" g="0.3" b="0.3" a="1.0"
                 x2="0" y2="-1.38778e-17" z2="-0.025" roll2="-1.5708" pitch2="-1.90898e-42" yaw2="4.22367e-17"/>
-    <gazebo reference="banh_xe_2">
-        <material>Gazebo/Gray</material>
-        <mu1>0.2</mu1>
-        <mu2>0.2</mu2>
-    </gazebo>
+    <xacro:gazebo reference="banh_xe_2" material="Gazebo/Gray" mu1="0.2" mu2="0.2"/>
     <xacro:joint joint_name="than_xe_banh_2" type="continuous"
                  x1="0.132437" y1="0.14" z1="0.0641321" roll1="-1.5708" pitch1="1.05145" yaw1="3.14159"
@@ -41,9 +33,5 @@
                 r="0.3" g="0.3" b="0.3" a="1.0"
                 x2="0" y2="3.46945e-18" z2="-0.025" roll2="-1.5708" pitch2="0" yaw2="-1.73484e-17"/>
-    <gazebo reference="banh_xe_3">
-        <material>Gazebo/Gray</material>
-        <mu1>0.2</mu1>
-        <mu2>0.2</mu2>
-    </gazebo>
+    <xacro:gazebo reference="banh_xe_3" material="Gazebo/Gray" mu1="0.2" mu2="0.2"/>
     <xacro:joint joint_name="than_xe_banh_3" type="continuous"
                  x1="-0.127563" y1="-0.14" z1="0.0641321" roll1="-1.5708" pitch1="0.295982" yaw1="0"
@@ -58,9 +46,5 @@
                 r="0.3" g="0.3" b="0.3" a="1.0"
                 x2="2.77556e-17" y2="0" z2="-0.025" roll2="-1.5708" pitch2="7.68415e-43" yaw2="1.4056e-18"/>
-    <gazebo reference="banh_xe_4">
-        <material>Gazebo/Gray</material>
-        <mu1>0.2</mu1>
-        <mu2>0.2</mu2>
-    </gazebo>
+    <xacro:gazebo reference="banh_xe_4" material="Gazebo/Gray" mu1="0.2" mu2="0.2"/>
     <xacro:joint joint_name="than_xe_banh_4" type="continuous"
                  x1="0.132437" y1="-0.14" z1="0.0641321" roll1="1.5708" pitch1="0.033338" yaw1="3.14159"
@@ -75,9 +59,5 @@
                 r="0.1" g="0.1" b="0.1" a="1.0"
                 x2="3.40439e-16" y2="-5.55112e-17" z2="0" roll2="1.5708" pitch2="0" yaw2="0"/>
-    <gazebo reference="xich_1">
-        <material>Gazebo/FlatBlack</material>
-        <mu1>0.2</mu1>
-        <mu2>0.2</mu2>
-    </gazebo>
+    <xacro:gazebo reference="xich_1" material="Gazebo/FlatBlack" mu1="0.2" mu2="0.2"/>
     <xacro:joint joint_name="than_xe_xich_1" type="fixed"
                  x1="0.0025" y1="-0.105" z1="0.064" roll1="-1.5708" pitch1="1.82546e-16" yaw1="0"
@@ -90,9 +70,5 @@
                 r="0.1" g="0.1" b="0.1" a="1.0"
                 x2="-0.0432788" y2="-0.055" z2="-0.06" roll2="-1.5708" pitch2="0" yaw2="0"/>
-    <gazebo reference="xich_2">
-        <material>Gazebo/FlatBlack</material>
-        <mu1>0.2</mu1>
-        <mu2>0.2</mu2>
-    </gazebo>
+    <xacro:gazebo reference="xich_2" material="Gazebo/FlatBlack" mu1="0.2" mu2="0.2"/>
     <xacro:joint joint_name="than_xe_xich_2" type="fixed"
                  x1="-0.0406" y1="0.105" z1="0.0091" roll1="-1.5708" pitch1="0" yaw1="3.14159"
@@ -117,3 +93,10 @@
         </plugin>
     </gazebo>
+    <gazebo>
+        <plugin name="gazebo_ros_control" filename="libgazebo_ros_control.so">
+            <robotNamespace>/xe_tang</robotNamespace>
+        </plugin>
+    </gazebo>
+    <xacro:transmission joint_name="than_xe_banh_4" actuator_name="left_wheel_motor"/>
+    <xacro:transmission joint_name="than_xe_banh_2" actuator_name="right_wheel_motor"/>
 </robot>

File: description/camera.xacro (robot description, xacro)
@@ -8,9 +8,5 @@
                 x2="1.9877e-18" y2="0" z2="0" roll2="3.14159" pitch2="0" yaw2="0"/>
     <link name="camera_optical"/>
-    <gazebo reference="camera">
-        <material>Gazebo/Green</material>
-        <mu1>0.2</mu1>
-        <mu2>0.2</mu2>
-    </gazebo>
+    <xacro:gazebo reference="camera" material="Gazebo/Green" mu1="0.2" mu2="0.2"/>
     <gazebo reference="camera_optical">
         <sensor name="camera" type="camera">

File: description/xe_tang.urdf.xacro (robot description, xacro)
@@ -1,4 +1,5 @@
 <?xml version="1.0"?>
 <robot xmlns:xacro="http://www.ros.org/wiki/xacro" name="xe-tang">
+    <xacro:property name="PI" value="3.141592653589793"/>
     <xacro:macro name="link" params="link_name
                                      x1 y1 z1 roll1 pitch1 yaw1
@@ -50,5 +51,23 @@
         </joint>
     </xacro:macro>
-    <xacro:property name="PI" value="3.141592653589793"/>
+    <xacro:macro name="transmission" params="joint_name actuator_name">
+        <transmission name="${joint_name}_transimission">
+            <type>transmission_interface/SimpleTransmission</type>
+            <actuator name="${actuator_name}">
+                <hardwareInterface>hardware_interface/EffortJointInterface</hardwareInterface>
+                <mechanicalReduction>1</mechanicalReduction>
+            </actuator>
+            <joint name="${joint_name}">
+                <hardwareInterface>hardware_interface/VelocityJointInterface</hardwareInterface>
+            </joint>
+        </transmission>
+    </xacro:macro>
+    <xacro:macro name="gazebo" params="reference material mu1 mu2">
+        <gazebo reference="${reference}">
+            <material>${material}</material>
+            <mu1>${mu1}</mu1>
+            <mu2>${mu2}</mu2>
+        </gazebo>
+    </xacro:macro>
     <xacro:link link_name="than_xe"
                 x1="0.00402455" y1="4.22475e-17" z1="0.0886727" roll1="0" pitch1="0" yaw1="0"
@@ -57,9 +76,5 @@
                 r="0.175" g="0.175" b="0.175" a="1.0"
                 x2="0.00243663" y2="4.16334e-17" z2="0.0391321" roll2="0" pitch2="0" yaw2="0"/>
-    <gazebo reference="than_xe">
-        <material>Gazebo/DarkGray</material>
-        <mu1>0.2</mu1>
-        <mu2>0.2</mu2>
-    </gazebo>
+    <xacro:gazebo reference="than_xe" material="Gazebo/DarkGray" mu1="0.2" mu2="0.2"/>
     <xacro:include filename="arm_controller.xacro"/>
     <xacro:include filename="base_controller.xacro"/>
