Commit message: v3.2.4

File: description/lidar.xacro (robot description, xacro)
@@ -17,8 +17,8 @@
                 <scan>
                     <horizontal>
-                        <samples>180</samples>
-                        <resolution>1.000000</resolution>
-                        <min_angle>1.5708</min_angle>
-                        <max_angle>${PI}</max_angle>
+                        <samples>360</samples>
+                        <resolution>1</resolution>
+                        <min_angle>-3.14</min_angle>
+                        <max_angle>3.14</max_angle>
                     </horizontal>
                 </scan>
@@ -26,5 +26,5 @@
                     <min>0.120000</min>
                     <max>3.5</max>
-                    <resolution>0.015000</resolution>
+                    <resolution>0.01</resolution>
                 </range>
                 <noise>

File: description/xe_tang.urdf.xacro (robot description, xacro)
@@ -1,5 +1,4 @@
 <?xml version="1.0"?>
 <robot xmlns:xacro="http://www.ros.org/wiki/xacro" name="xe-tang">
-    <xacro:property name="PI" value="3.141592653589793"/>
     <xacro:macro name="link" params="link_name
                                      x1 y1 z1 roll1 pitch1 yaw1
