Commit message: v.1.2.0

File: description/arm_controller.xacro (robot description, xacro)
@@ -13,6 +13,5 @@
                  x1="-0.173402" y1="0.0727514" z1="0.243141" roll1="3.14159" pitch1="0" yaw1="0"
                  parent_link="than_xe"
-                 child_link="khau_1"
-                 x2="0" y2="0" z2="1"/>
+                 child_link="khau_1"/>
     <xacro:link link_name="khop"
                 x1="7.82984e-19" y1="4.06082e-18" z1="-0.015" roll1="0" pitch1="0" yaw1="0"

File: description/base_controller.xacro (robot description, xacro)
@@ -73,6 +73,5 @@
                  x1="-0.235839" y1="-0.0322486" z1="0.169009" roll1="-1.5708" pitch1="0" yaw1="0"
                  parent_link="than_xe"
-                 child_link="xich_1"
-                 x2="0" y2="0" z2="1"/>
+                 child_link="xich_1"/>
     <xacro:link link_name="xich_2"
                 x1="-0.0432788" y1="-0.055" z1="-0.03" roll1="0" pitch1="0" yaw1="0"
@@ -87,5 +86,29 @@
                  x1="-0.278939" y1="0.177751" z1="0.114109" roll1="-1.5708" pitch1="0" yaw1="3.14159"
                  parent_link="than_xe"
-                 child_link="xich_2"
-                 x2="0" y2="0" z2="1"/>
+                 child_link="xich_2"/>
+    <transmission name="tran_left_wheel">
+        <type>transmission_interface/SimpleTransmission</type>
+        <joint name="than_xe_banh_1">
+        <hardwareInterface>hardware_interface/VelocityJointInterface</hardwareInterface>
+        </joint>
+        <actuator name="left_wheel_motor">
+        <hardwareInterface>hardware_interface/VelocityJointInterface</hardwareInterface>
+        <mechanicalReduction>1</mechanicalReduction>
+        </actuator>
+    </transmission>
+    <transmission name="tran_right_wheel">
+        <type>transmission_interface/SimpleTransmission</type>
+        <joint name="than_xe_banh_2">
+        <hardwareInterface>hardware_interface/VelocityJointInterface</hardwareInterface>
+        </joint>
+        <actuator name="right_wheel_motor">
+        <hardwareInterface>hardware_interface/VelocityJointInterface</hardwareInterface>
+        <mechanicalReduction>1</mechanicalReduction>
+        </actuator>
+    </transmission>
+    <gazebo>
+        <plugin name="gazebo_ros_control" filename="libgazebo_ros_control.so">
+        <robotNamespace>/xe_tang</robotNamespace>
+        </plugin>
+    </gazebo>
 </robot>

File: description/encoder.xacro (robot description, xacro)
@@ -13,7 +13,13 @@
 			<odometryFrame>odom</odometryFrame>
 			<robotBaseFrame>than_xe</robotBaseFrame>
-      		<publish_odom>true</publish_odom>
+			<publishTf>true</publishTf>
       		<publishOdomTF>true</publishOdomTF>
       		<publishWheelTF>true</publishWheelTF>
+			<rosDebugLevel>INFO</rosDebugLevel>
+			<publishWheelJointState>true</publishWheelJointState>
+			<wheelAcceleration>1.0</wheelAcceleration>
+			<wheelTorque>10</wheelTorque>
+			<updateRate>100</updateRate>
+			<odometrySource>encoder</odometrySource>
     	</plugin>
   	</gazebo>

File: description/xe_tang.urdf.xacro (robot description, xacro)
@@ -34,5 +34,5 @@
                                       parent_link
                                       child_link
-                                      x2 y2 z2
+                                      x2:=0 y2:=0 z2:=0
                                       effort:=0 velocity:=0 lower:=0 upper:=0">
         <joint name="${joint_name}" type="${type}">
@@ -40,10 +40,11 @@
             <parent link="${parent_link}"/>
             <child link="${child_link}"/>
-            <axis xyz="${x2} ${y2} ${z2}"/>
             <xacro:if value="${type == 'revolute' or type == 'prismatic'}">
+                <axis xyz="${x2} ${y2} ${z2}"/>
                 <limit effort="${effort}" velocity="${velocity}" lower="${lower}" upper="${upper}"/>
             </xacro:if>
         </joint>
     </xacro:macro>
+    <link name="world"/>
     <xacro:link link_name="than_xe"
                 x1="-0.234314" y1="0.0727514" z1="0.193682" roll1="0" pitch1="0" yaw1="0"
@@ -55,4 +56,8 @@
         <material>Gazebo/DarkGray</material>
     </gazebo>
+    <xacro:joint joint_name="world_than_xe" type="fixed"
+                 x1="0" y1="0" z1="0" roll1="0" pitch1="0" yaw1="0"
+                 parent_link="world"
+                 child_link="than_xe"/>
     <xacro:include filename="arm_controller.xacro"/>
     <xacro:include filename="base_controller.xacro"/>

Commit message: v1.3.8

File: description/arm_controller.xacro (robot description, xacro)
@@ -7,9 +7,5 @@
                 r="1.0" g="1.0" b="1.0" a="1.0"
                 x2="0" y2="3.33585e-18" z2="0" roll2="3.14159" pitch2="0" yaw2="0"/>
-    <gazebo reference="khau_1">
-        <material>Gazebo/White</material>
-        <mu1>0.2</mu1>
-        <mu2>0.2</mu2>
-    </gazebo>
+    <xacro:gazebo reference="khau_1" material="Gazebo/White" mu1="0.2" mu2="0.2"/>
     <xacro:joint joint_name="than_xe_khau_1" type="fixed"
                  x1="0.0649366" y1="4.67039e-17" z1="0.138132" roll1="3.14159" pitch1="0" yaw1="0"
@@ -22,15 +18,10 @@
                 r="0.13" g="0.44" b="0.70" a="1.0"
                 x2="0" y2="-3.9801e-18" z2="-0.03" roll2="0" pitch2="0" yaw2="1.3617e-45"/>
-    <gazebo reference="khop">
-        <material>Gazebo/SkyBlue</material>
-        <mu1>0.2</mu1>
-        <mu2>0.2</mu2>
-    </gazebo>
+    <xacro:gazebo reference="khop" material="Gazebo/SkyBlue" mu1="0.2" mu2="0.2"/>
     <xacro:joint joint_name="khau_1_khop" type="prismatic"
                  x1="0" y1="2.80737e-25" z1="-0.210059" roll1="-3.14159" pitch1="6.59901e-17" yaw1="-1.96037e-29"
                  parent_link="khau_1"
                  child_link="khop"
-                 x2="0" y2="0" z2="1"
-                 effort="10" velocity="10" lower="-0.135059" upper="0.234941"/>
+                 x2="0" y2="0" z2="1" effort="10" velocity="10" lower="-0.135059" upper="0.234941"/>
     <xacro:link link_name="khau_2"
                 x1="0.228819" y1="-6.22477e-10" z1="-0.0150176" roll1="0" pitch1="0" yaw1="0"
@@ -39,14 +30,9 @@
                 r="1.0" g="1.0" b="1.0" a="1.0"
                 x2="0" y2="-3.90313e-18" z2="-0.03" roll2="-5.99742e-33" pitch2="-6.51514e-33" yaw2="-3.10412e-18"/>
-    <gazebo reference="khau_2">
-        <material>Gazebo/White</material>
-        <mu1>0.2</mu1>
-        <mu2>0.2</mu2>
-    </gazebo>
+    <xacro:gazebo reference="khau_2" material="Gazebo/White" mu1="0.2" mu2="0.2"/>
     <xacro:joint joint_name="khop_khau_2" type="revolute"
                  x1="0" y1="8.97939e-27" z1="0" roll1="-9.25178e-17" pitch1="2.59191e-16" yaw1="-3.12038"
                  parent_link="khop"
                  child_link="khau_2"
-                 x2="0" y2="0" z2="1"
-                 effort="10" velocity="10" lower="-3.141592653589793" upper="3.141592653589793"/>
+                 x2="0" y2="0" z2="1" effort="10" velocity="10" lower="-${PI}" upper="${PI}"/>
 </robot>

File: description/base_controller.xacro (robot description, xacro)
@@ -12,6 +12,5 @@
                  parent_link="than_xe"
                  child_link="banh_xe_1"
-                 x2="0" y2="0" z2="1"
-                 effort="10" velocity="10"/>
+                 x2="0" y2="0" z2="1" effort="10" velocity="10"/>
     <xacro:link link_name="banh_xe_2"
                 x1="-1.63473e-19" y1="-9.18731e-18" z1="0.00430301" roll1="0" pitch1="0" yaw1="0"
@@ -25,6 +24,5 @@
                  parent_link="than_xe"
                  child_link="banh_xe_2"
-                 x2="0" y2="0" z2="1"
-                 effort="10" velocity="10"/>
+                 x2="0" y2="0" z2="1" effort="10" velocity="10"/>
     <xacro:link link_name="banh_xe_3"
                 x1="-1.63473e-19" y1="8.15992e-18" z1="0.00430301" roll1="0" pitch1="0" yaw1="0"
@@ -38,6 +36,5 @@
                  parent_link="than_xe"
                  child_link="banh_xe_3"
-                 x2="0" y2="0" z2="1"
-                 effort="10" velocity="10"/>
+                 x2="0" y2="0" z2="1" effort="10" velocity="10"/>
     <xacro:link link_name="banh_xe_4"
                 x1="2.75921e-17" y1="4.69047e-18" z1="0.00430301" roll1="0" pitch1="0" yaw1="0"
@@ -51,6 +48,5 @@
                  parent_link="than_xe"
                  child_link="banh_xe_4"
-                 x2="0" y2="0" z2="1"
-                 effort="10" velocity="10"/>
+                 x2="0" y2="0" z2="1" effort="10" velocity="10"/>
     <xacro:link link_name="xich_1"
                 x1="3.10096e-16" y1="-4.79297e-17" z1="-0.03" roll1="0" pitch1="0" yaw1="0"

File: description/xe_tang.urdf.xacro (robot description, xacro)
@@ -70,4 +70,5 @@
         </gazebo>
     </xacro:macro>
+    <!-- ~~~~~~~~~~~~~~~~~~~~~~~~~~~~~~~~~~~~~~~~~~ -->
     <xacro:link link_name="than_xe"
                 x1="0.00402455" y1="4.22475e-17" z1="0.0886727" roll1="0" pitch1="0" yaw1="0"

Commit message: v.3.1.4

File: description/arm_controller.xacro (robot description, xacro)
@@ -39,5 +39,5 @@
         <robotNamespace>/</robotNamespace>
     </plugin>
-    <xacro:transmission joint_name="khop_joint" actuator_name="lower_motor"/>
-    <xacro:transmission joint_name="khau_2_joint" actuator_name="upper_motor"/>
+    <xacro:arm_transmission joint_name="khop_joint" actuator_name="lower_motor"/>
+    <xacro:arm_transmission joint_name="khau_2_joint" actuator_name="upper_motor"/>
 </robot>

File: description/base_controller.xacro (robot description, xacro)
@@ -76,7 +76,7 @@
         </plugin>
     </gazebo>
-    <xacro:transmission joint_name="banh_xe_4_joint" actuator_name="left_wheel_motor"/>
-    <xacro:transmission joint_name="banh_xe_3_joint" actuator_name="left_wheel_motor"/>
-    <xacro:transmission joint_name="banh_xe_2_joint" actuator_name="right_wheel_motor"/>
-    <xacro:transmission joint_name="banh_xe_1_joint" actuator_name="left_wheel_motor"/>
+    <xacro:base_transmission joint_name="banh_xe_4_joint" actuator_name="left_wheel_motor"/>
+    <xacro:base_transmission joint_name="banh_xe_3_joint" actuator_name="left_wheel_motor"/>
+    <xacro:base_transmission joint_name="banh_xe_2_joint" actuator_name="right_wheel_motor"/>
+    <xacro:base_transmission joint_name="banh_xe_1_joint" actuator_name="left_wheel_motor"/>
 </robot>

File: description/xe_tang.urdf.xacro (robot description, xacro)
@@ -51,5 +51,5 @@
         </joint>
     </xacro:macro>
-    <xacro:macro name="transmission" params="joint_name actuator_name">
+    <xacro:macro name="base_transmission" params="joint_name actuator_name">
         <transmission name="${joint_name}_transmission">
             <type>transmission_interface/SimpleTransmission</type>
@@ -60,4 +60,16 @@
             <joint name="${joint_name}">
                 <hardwareInterface>hardware_interface/VelocityJointInterface</hardwareInterface>
+            </joint>
+        </transmission>
+    </xacro:macro>
+    <xacro:macro name="arm_transmission" params="joint_name actuator_name">
+        <transmission name="${joint_name}_transmission">
+            <type>transmission_interface/SimpleTransmission</type>
+            <actuator name="${actuator_name}">
+                <hardwareInterface>hardware_interface/EffortJointInterface</hardwareInterface>
+                <mechanicalReduction>1</mechanicalReduction>
+            </actuator>
+            <joint name="${joint_name}">
+                <hardwareInterface>hardware_interface/EffortJointInterface</hardwareInterface>
             </joint>
         </transmission>

Commit message: v3.1.5

File: description/arm_controller.xacro (robot description, xacro)
@@ -31,13 +31,13 @@
                 x2="0" y2="-3.90313e-18" z2="-0.03" roll2="-5.99742e-33" pitch2="-6.51514e-33" yaw2="-3.10412e-18"/>
     <xacro:gazebo reference="khau_2" material="Gazebo/White" mu1="0.2" mu2="0.2"/>
-    <xacro:joint joint_name="khau_2_joint" type="revolute"
+    <xacro:joint joint_name="khau_2_joint" type="continuous"
                  x1="0" y1="8.97939e-27" z1="0" roll1="-9.25178e-17" pitch1="2.59191e-16" yaw1="-3.12038"
                  parent_link="khop"
                  child_link="khau_2"
-                 x2="0" y2="0" z2="1" effort="10" velocity="10" lower="-${PI}" upper="${PI}"/>
+                 x2="0" y2="0" z2="1" effort="10" velocity="10"/>
     <plugin name="arm_control" filename="libgazebo_ros_control.so">
         <robotNamespace>/</robotNamespace>
     </plugin>
-    <xacro:arm_transmission joint_name="khop_joint" actuator_name="lower_motor"/>
-    <xacro:arm_transmission joint_name="khau_2_joint" actuator_name="upper_motor"/>
+    <xacro:arm_transmission joint_name="khop_joint" actuator_name="lower_motor" hwInterface="hardware_interface/VelocityJointInterface"/>
+    <xacro:arm_transmission joint_name="khau_2_joint" actuator_name="upper_motor" hwInterface="hardware_interface/EffortJointInterface"/>
 </robot>

File: description/xe_tang.urdf.xacro (robot description, xacro)
@@ -63,13 +63,13 @@
         </transmission>
     </xacro:macro>
-    <xacro:macro name="arm_transmission" params="joint_name actuator_name">
+    <xacro:macro name="arm_transmission" params="joint_name actuator_name hwInterface">
         <transmission name="${joint_name}_transmission">
             <type>transmission_interface/SimpleTransmission</type>
             <actuator name="${actuator_name}">
-                <hardwareInterface>hardware_interface/EffortJointInterface</hardwareInterface>
+                <hardwareInterface>${hwInterface}</hardwareInterface>
                 <mechanicalReduction>1</mechanicalReduction>
             </actuator>
             <joint name="${joint_name}">
-                <hardwareInterface>hardware_interface/EffortJointInterface</hardwareInterface>
+                <hardwareInterface>${hwInterface}</hardwareInterface>
             </joint>
         </transmission>

Commit message: v3.2.2

File: description/arm_controller.xacro (robot description, xacro)
@@ -39,5 +39,5 @@
         <robotNamespace>/</robotNamespace>
     </plugin>
-    <xacro:arm_transmission joint_name="khop_joint" actuator_name="lower_motor" hwInterface="hardware_interface/EffortJointInterface"/>
-    <xacro:arm_transmission joint_name="khau_2_joint" actuator_name="upper_motor" hwInterface="hardware_interface/EffortJointInterface"/>
+    <xacro:arm_transmission joint_name="khop_joint" actuator_name="lower_motor"/>
+    <xacro:arm_transmission joint_name="khau_2_joint" actuator_name="upper_motor"/>
 </robot>

File: description/xe_tang.urdf.xacro (robot description, xacro)
@@ -63,13 +63,13 @@
         </transmission>
     </xacro:macro>
-    <xacro:macro name="arm_transmission" params="joint_name actuator_name hwInterface">
+    <xacro:macro name="arm_transmission" params="joint_name actuator_name">
         <transmission name="${joint_name}_transmission">
             <type>transmission_interface/SimpleTransmission</type>
             <actuator name="${actuator_name}">
-                <hardwareInterface>${hwInterface}</hardwareInterface>
+                <hardwareInterface>hardware_interface/EffortJointInterface</hardwareInterface>
                 <mechanicalReduction>1</mechanicalReduction>
             </actuator>
             <joint name="${joint_name}">
-                <hardwareInterface>${hwInterface}</hardwareInterface>
+                <hardwareInterface>hardware_interface/EffortJointInterface</hardwareInterface>
             </joint>
         </transmission>
